Commit message: Upgrade robot from 2D to 3D 4DOF

File: sketch_follower/robot_description/urdf/2d_2dof.xacro (robot description, xacro)
@@ -11,5 +11,5 @@
             <origin xyz="0.0 0.0 0.0" rpy="0 0.0 0.0"/>
             <geometry>
-                 <mesh filename="package://sketch_follower/robot_description/meshes/base_link.stl" scale="${sf} ${sf} ${sf}"/>
+                 <mesh filename="package://sketch_follower/robot_description/meshes/2d_base_link.stl" scale="${sf} ${sf} ${sf}"/>
             </geometry>
             <material name="blue" />
@@ -18,5 +18,5 @@
             <origin xyz="0.0 0.0 0.0" rpy="0.0 0.0 0.0"/>
             <geometry>
-                 <mesh filename="package://sketch_follower/robot_description/meshes/base_link.stl" scale="${sf} ${sf} ${sf}"/>
+                 <mesh filename="package://sketch_follower/robot_description/meshes/2d_base_link.stl" scale="${sf} ${sf} ${sf}"/>
             </geometry>
         </collision>

File: sketch_follower/robot_description/urdf/2d_3dof.xacro (robot description, xacro)
@@ -11,5 +11,5 @@
             <origin xyz="0.0 0.0 0.0" rpy="0 0.0 0.0"/>
             <geometry>
-                 <mesh filename="package://sketch_follower/robot_description/meshes/base_link.stl" scale="${sf} ${sf} ${sf}"/>
+                 <mesh filename="package://sketch_follower/robot_description/meshes/2d_base_link.stl" scale="${sf} ${sf} ${sf}"/>
             </geometry>
             <material name="blue" />
@@ -18,5 +18,5 @@
             <origin xyz="0.0 0.0 0.0" rpy="0.0 0.0 0.0"/>
             <geometry>
-                 <mesh filename="package://sketch_follower/robot_description/meshes/base_link.stl" scale="${sf} ${sf} ${sf}"/>
+                 <mesh filename="package://sketch_follower/robot_description/meshes/2d_base_link.stl" scale="${sf} ${sf} ${sf}"/>
             </geometry>
         </collision>

File: sketch_follower/robot_description/urdf/helpers.xacro (robot description, xacro)
@@ -20,5 +20,5 @@
                 <origin xyz="0 0.0 0.0" rpy="0.0 0.0 0.0"/>
                 <geometry>
-                    <mesh filename="package://sketch_follower/robot_description/meshes/link.stl" scale="${sf} ${sf} ${sf}"/>
+                    <mesh filename="package://sketch_follower/robot_description/meshes/2d_link.stl" scale="${sf} ${sf} ${sf}"/>
                 </geometry>
                 <material name="${material}" />
@@ -27,5 +27,5 @@
                 <origin xyz="0.0 0.0 0.0" rpy="0.0 0.0 0.0"/>
                 <geometry>
-                    <mesh filename="package://sketch_follower/robot_description/meshes/link.stl" scale="${sf} ${sf} ${sf}"/>
+                    <mesh filename="package://sketch_follower/robot_description/meshes/2d_link.stl" scale="${sf} ${sf} ${sf}"/>
                 </geometry>
             </collision>
