Commit message: Fix display issues

File: robot_description/urdf/helpers.xacro (robot description, xacro)
@@ -1,5 +1,4 @@
 <?xml version="1.0"?>
 <robot xmlns:xacro="http://www.ros.org/wiki/xacro">
-    <xacro:property name="sf" value="0.005"/>
     <material name="blue">
         <color rgba="0 0.5 1 1" />

Commit message: Create launch file with Rviz and ROS 2 control

File: robot_description/urdf/helpers.xacro (robot description, xacro)
@@ -1,5 +1,4 @@
 <?xml version="1.0"?>
 <robot xmlns:xacro="http://www.ros.org/wiki/xacro">
-    <xacro:property name="sf" value="0.005"/>
     <material name="blue">
         <color rgba="0 0.5 1 1" />
@@ -41,16 +40,3 @@
         </inertial>
     </xacro:macro>
-    <xacro:macro name="transmission" params="name">
-        <transmission name='${name}_transmission'>
-            <type>transmission_interface/SimpleTransmission</type>
-                <joint name='${name}'>
-                    <hardwareInterface>hardware_interface/VelocityJointInterface</hardwareInterface>
-                </joint>
-            <actuator name='${name}_actuator'>
-                <hardwareInterface>hardware_interface/VelocityJointInterface</hardwareInterface>
-                <mechanicalReduction>1</mechanicalReduction>
-            </actuator>
-        </transmission>
-    </xacro:macro>
-    <!-- EffortJointInterface -->
 </robot>

File: robot_description/urdf/model.xacro (robot description, xacro)
@@ -1,9 +1,8 @@
 <?xml version="1.0"?>
-<robot xmlns:xacro="http://www.ros.org/wiki/xacro" name="sketch_follower_3d_4dof">
+<robot xmlns:xacro="http://www.ros.org/wiki/xacro" name="sketch_follower">
     <xacro:include filename="$(find sketch_follower)/robot_description/urdf/helpers.xacro"/>
+    <xacro:include filename="$(find sketch_follower)/robot_description/urdf/ros2_control.xacro"/>
+    <xacro:sketch_follower_ros2_control/>
     <xacro:property name="sf" value="0.02"/>
-    <gazebo>
-        <plugin filename="libgazebo_ros_control.so" name="gazebo_ros_control" />
-    </gazebo>
     <link name="world" />
     <link name="base">
@@ -23,7 +22,4 @@
         </collision>
     </link>
-    <gazebo reference="base">
-        <material>Gazebo/White</material>
-    </gazebo>
     <joint name="base_joint" type="fixed">
         <origin xyz="0.0 0.0 0" rpy="0.0 0.0 0"/>
@@ -47,15 +43,11 @@
         </collision>
     </link>
-    <gazebo reference="base_arm_slot">
-        <material>Gazebo/Black</material>
-    </gazebo>
     <joint name="base_arm_slot_joint" type="continuous">
         <origin xyz="0.0 0.0 0.6" rpy="0.0 0.0 0.0"/>
         <parent link="base"/>
         <child link="base_arm_slot"/>
-        <axis xyz="0.0 0.0 1.0"/>
+        <axis xyz="0 0 1"/>
         <dynamics damping="2.0" friction="2.0"/>
     </joint>
-    <xacro:transmission name="base_arm_slot_joint" />
     <link name="arm_link_1">
         <xacro:inertial m="1.2" x="0.7" y="0.4" z="2" oy="0" oz="1" />
@@ -74,15 +66,11 @@
         </collision>
     </link>
-    <gazebo reference="arm_link_1">
-        <material>Gazebo/White</material>
-    </gazebo>
     <joint name="arm_link_1_joint" type="continuous">
         <origin xyz="0.0 -0.1 0.8" rpy="0.0 0.0 0.0"/>
         <parent link="base_arm_slot"/>
         <child link="arm_link_1"/>
-        <axis xyz="0.0 1.0 0.0"/>
+        <axis xyz="0 1 0"/>
         <dynamics damping="2.0" friction="2.0"/>
     </joint>
-    <xacro:transmission name="arm_link_1_joint" />
     <link name="arm_link_2">
         <xacro:inertial m="1.2" x="0.7" y="0.4" z="2" oy="0" oz="1" />
@@ -101,15 +89,11 @@
         </collision>
     </link>
-    <gazebo reference="arm_link_2">
-        <material>Gazebo/Black</material>
-    </gazebo>
     <joint name="arm_link_2_joint" type="continuous">
         <origin xyz="0.0 0.4 2.0" rpy="0.0 0.0 0.0"/>
         <parent link="arm_link_1"/>
         <child link="arm_link_2"/>
-        <axis xyz="0.0 1.0 0.0"/>
+        <axis xyz="0 1 0"/>
         <dynamics damping="2.0" friction="2.0"/>
     </joint>
-    <xacro:transmission name="arm_link_2_joint" />
     <link name="end_effector">
         <xacro:inertial m="1.2" x="1" y="0.4" z="1" oy="0" oz="0.5" />
@@ -128,14 +112,10 @@
         </collision>
     </link>
-    <gazebo reference="end_effector">
-        <material>Gazebo/White</material>
-    </gazebo>
     <joint name="end_effector_joint" type="continuous">
         <origin xyz="0.0 -0.4 2.0" rpy="0.0 0.0 0.0"/>
         <parent link="arm_link_2"/>
         <child link="end_effector"/>
-        <axis xyz="0.0 1.0 0.0"/>
+        <axis xyz="0 1 0"/>
         <dynamics damping="2.0" friction="2.0"/>
     </joint>
-    <xacro:transmission name="end_effector_joint" />
 </robot>
